Commit message: updated oak d config and xacro

File: src/ugv_with_arm_camera_description/urdf/components/oak_d_pro.urdf.xacro (robot description, xacro)
@@ -1,5 +1,5 @@
 <?xml version="1.0"?>
 <robot xmlns:xacro="http://www.ros.org/wiki/xacro" name="oak_d_pro">
-<xacro:macro name="oak_d_pro" params="prefix:='camera_' parent origin_xyz origin_rpy">
+<xacro:macro name="oak_d_pro" params="prefix:='oak_d_pro_' parent origin_xyz origin_rpy">
   <joint name="${prefix}joint" type="fixed">
     <parent link="${parent}"/>
