Commit message: seperated perception from the rpi5

File: src/ugv_with_arm_camera_description/urdf/components/ugv_rover_base.urdf.xacro (robot description, xacro)
@@ -1,5 +1,5 @@
 <?xml version="1.0"?>
 <robot xmlns:xacro="http://www.ros.org/wiki/xacro" name="ugv_rover_base">
-<xacro:macro name="ugv_rover_base" params="prefix:=''">
+<xacro:macro name="ugv_rover_base" params="prefix:='' wheel_joint_type:='continuous'">
   <link name="${prefix}base_footprint"/>
   <joint name="${prefix}base_joint" type="fixed">
@@ -34,5 +34,5 @@
   <link name="${prefix}base_imu_link"/>
   <!-- Left front wheel -->
-  <joint name="${prefix}left_up_wheel_joint" type="continuous">
+  <joint name="${prefix}left_up_wheel_joint" type="${wheel_joint_type}">
     <origin xyz="0.0855 0.08726 -0.041212" rpy="1.5708 0 0"/>
     <parent link="${prefix}base_link"/>
@@ -60,5 +60,5 @@
   </link>
   <!-- Left rear wheel -->
-  <joint name="${prefix}left_down_wheel_joint" type="continuous">
+  <joint name="${prefix}left_down_wheel_joint" type="${wheel_joint_type}">
     <origin xyz="-0.0855 0.08726 -0.041212" rpy="1.5708 0 0"/>
     <parent link="${prefix}base_link"/>
@@ -86,5 +86,5 @@
   </link>
   <!-- Right front wheel -->
-  <joint name="${prefix}right_up_wheel_joint" type="continuous">
+  <joint name="${prefix}right_up_wheel_joint" type="${wheel_joint_type}">
     <origin xyz="0.0855 -0.08726 -0.041212" rpy="1.5708 0 0"/>
     <parent link="${prefix}base_link"/>
@@ -112,5 +112,5 @@
   </link>
   <!-- Right rear wheel -->
-  <joint name="${prefix}right_down_wheel_joint" type="continuous">
+  <joint name="${prefix}right_down_wheel_joint" type="${wheel_joint_type}">
     <origin xyz="-0.0855 -0.08726 -0.041212" rpy="1.5708 0 0"/>
     <parent link="${prefix}base_link"/>
